Commit message: 匹配URDF和控制器参数
- 更新URDF质量到12kg（真实Lite3重量）
- 更新控制器惯性矩参数：Ib_从[0.0792,0.2085,0.2265]改为[0.07416,0.12086,0.15067]
- 更新控制器质心偏移：pcb_从[0,0,0]改为[0.00160,-0.00039,-0.01164]
- 更新摩擦系数：从0.4改为0.6以匹配URDF
- 修复leg.xacro中缺失的</mass>标签
- 验证参数匹配性和系统启动

File: lite3_description/urdf/robot.urdf (robot description, URDF)
Before this commit: robot lite3, 20 links, 19 joints
Links:
- removed link INERTIA
- link FL_FOOT: mass 1E-12 -> 0.08179029876178574
- link FL_HIP: mass 0.428 -> 0.5834374645007383; geometry visual mesh filename=file:///home/longkang/quadruped_ws/install/lite3_descriptio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
- link FL_SHANK: mass 0.115 -> 0.1567647392934227; geometry collision box size=0.02 0.02 0.18; visual mesh filename=file:///home/longkang/quadruped_ws/install/lite3_descriptio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
- link FL_THIGH: mass 0.61 -> 0.8315347040781551; geometry collision box size=0.02 0.02 0.16; visual mesh filename=file:///home/longkang/quadruped_ws/install/lite3_descriptio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
- link FR_FOOT: mass 1E-12 -> 0.08179029876178574
- link FR_HIP: mass 0.428 -> 0.5834374645007383; geometry visual mesh filename=file:///home/longkang/quadruped_ws/install/lite3_descriptio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
- link FR_SHANK: mass 0.115 -> 0.1567647392934227; geometry collision box size=0.02 0.02 0.18; visual mesh filename=file:///home/longkang/quadruped_ws/install/lite3_descriptio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
- link FR_THIGH: mass 0.61 -> 0.8315347040781551; geometry collision box size=0.02 0.02 0.16; visual mesh filename=file:///home/longkang/quadruped_ws/install/lite3_descriptio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
- link HL_FOOT: mass 1E-12 -> 0.08179029876178574
- link HL_HIP: mass 0.428 -> 0.5834374645007383; geometry visual mesh filename=file:///home/longkang/quadruped_ws/install/lite3_descriptio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
- link HL_SHANK: mass 0.115 -> 0.1567647392934227; geometry collision box size=0.02 0.02 0.18; visual mesh filename=file:///home/longkang/quadruped_ws/install/lite3_descriptio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
- link HL_THIGH: mass 0.61 -> 0.8315347040781551; geometry collision box size=0.02 0.02 0.16; visual mesh filename=file:///home/longkang/quadruped_ws/install/lite3_descriptio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
- link HR_FOOT: mass 1E-12 -> 0.08179029876178574
- link HR_HIP: mass 0.428 -> 0.5834374645007383; geometry visual mesh filename=file:///home/longkang/quadruped_ws/install/lite3_descriptio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
- link HR_SHANK: mass 0.115 -> 0.1567647392934227; geometry collision box size=0.02 0.02 0.18; visual mesh filename=file:///home/longkang/quadruped_ws/install/lite3_descriptio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
- link HR_THIGH: mass 0.61 -> 0.8315347040781551; geometry collision box size=0.02 0.02 0.16; visual mesh filename=file:///home/longkang/quadruped_ws/install/lite3_descriptio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
- link TORSO: mass None -> 5.629898899102925; geometry collision box size=0.35 0.184 0.08; visual mesh filename=file:///home/longkang/quadruped_ws/install/lite3_descriptio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
Joints:
- removed joint Torso2Inertia
- joint FL_HipX: origin xyz=0.1745 0.062 0 -> xyz=0.1745 0.062 0 rpy=0 0 0
- joint FL_HipY: origin xyz=0 0.0985 0 -> xyz=0 0.0955 0
- joint FR_HipX: origin xyz=0.1745 -0.062 0 -> xyz=0.1745 -0.062 0 rpy=0 0 0
- joint FR_HipY: origin xyz=0 -0.0985 0 -> xyz=0 -0.0955 0
- joint HL_HipX: origin xyz=-0.1745 0.062 0 -> xyz=-0.1745 0.062 0 rpy=0 0 0
- joint HL_HipY: origin xyz=0 0.0985 0 -> xyz=0 0.0955 0
- joint HR_HipX: origin xyz=-0.1745 -0.062 0 -> xyz=-0.1745 -0.062 0 rpy=0 0 0
- joint HR_HipY: origin xyz=0 -0.0985 0 -> xyz=0 -0.0955 0

File: lite3_description/xacro/leg.xacro (robot description, xacro)
@@ -86,6 +86,6 @@
       <inertial>
         <origin xyz="0.00585 -8.732E-07 -0.12"/>
-        <mass value="0.115"/>
-        <inertia ixx="6.68E-04" ixy="-1.24E-08" ixz="6.91E-06" iyy="6.86E-04" iyz="5.65E-09" izz="3.155E-05"/>
+        <mass value="0.1567647392934227"></mass>
+        <inertia ixx="9.104550629239001e-04" ixy="-1.690647476476001e-08" ixz="9.41971624706656e-06" iyy="9.353157488964166e-04" iyz="7.70211998592336e-09" izz="4.30081045672405e-05"/>
       </inertial>
       <visual>

File: lite3_description/xacro/robot.xacro (robot description, xacro)
@@ -43,7 +43,7 @@
     <inertial>
       <origin xyz="0.004098 -0.000663 -0.002069"/>
-      <mass value="4.130"/>
-      <inertia ixx="0.016982120" ixy="2.1294E-05" ixz="6.0763E-05" iyy="0.030466501" iyz="1.7968E-05"
-               izz="0.042609956"/>
+      <mass value="5.629898899102925"/>
+      <inertia ixx="0.023148999999999998" ixy="2.9029999999999997e-05" ixz="8.283e-05" iyy="0.041535" iyz="2.449e-05"
+               izz="0.058079999999999996"/>
     </inertial>
   </link>
@@ -57,5 +57,5 @@
       <mass value="0.001"/>
       <origin rpy="0 0 0" xyz="0 0 0"/>
-      <inertia ixx="0.0001" ixy="0" ixz="0" iyy="0.0001" iyz="0" izz="0.0001"/>
+      <inertia ixx="0.02938701137712478" ixy="2.9029999999999997e-05" ixz="8.283e-05" iyy="0.05272752678512583" iyz="2.449e-05" izz="0.07373094391910696"/>
     </inertial>
     <visual>

Commit message: feat: 添加了xacro2controller参数自动适配

File: lite3_description/urdf/robot.urdf (robot description, URDF)
Before this commit: robot lite3, 19 links, 18 joints
Links:
- link FL_FOOT: mass 0.08179029876178574 -> 0.01519029876178574
- link FR_FOOT: mass 0.08179029876178574 -> 0.01519029876178574
- link HL_FOOT: mass 0.08179029876178574 -> 0.01519029876178574
- link HR_FOOT: mass 0.08179029876178574 -> 0.01519029876178574
