Commit message: Refactor Gazebo Classic world assets

File: libraries/quadruped_playground/models/D435/model.xacro (robot description, xacro)
@@ -22,5 +22,5 @@
         <origin xyz="0 0 0" rpy="0 0 1.57"/>
         <geometry>
-          <mesh filename="file://$(find gz_quadruped_playground)/models/D435/meshes/realsense.dae" scale="1 1 1"/>
+          <mesh filename="file://$(find quadruped_playground)/models/D435/meshes/realsense.dae" scale="1 1 1"/>
         </geometry>
       </visual>

File: libraries/quadruped_playground/models/Lidar3DV1/model.xacro (robot description, xacro)
@@ -21,5 +21,5 @@
       <visual>
         <geometry>
-          <mesh filename="file://$(find gz_quadruped_playground)/models/Lidar3DV1/meshes/lidar_3d_v1.dae" scale="1 1 1"/>
+          <mesh filename="file://$(find quadruped_playground)/models/Lidar3DV1/meshes/lidar_3d_v1.dae" scale="1 1 1"/>
         </geometry>
       </visual>

File: lite3_description/xacro/gazebo.xacro (robot description, xacro)
@@ -240,6 +240,6 @@
   <xacro:arg name="EXTERNAL_SENSORS" default="false"/>
   <xacro:if value="$(arg EXTERNAL_SENSORS)">
-    <xacro:include filename="$(find gz_quadruped_playground)/models/D435/model.xacro"/>
-    <xacro:include filename="$(find gz_quadruped_playground)/models/Lidar3DV1/model.xacro"/>
+    <xacro:include filename="$(find quadruped_playground)/models/D435/model.xacro"/>
+    <xacro:include filename="$(find quadruped_playground)/models/Lidar3DV1/model.xacro"/>
     <xacro:d435 camID="1" name="d435">
       <origin rpy="0 0.1 0" xyz="0.23 0 0.06"/>
